File: V1/relay-24v-4ch-8a-v1.kicad_sch (KiCad schematic)
At the start: 24 parts, among them J1 250-202, J2 250-204, J3 DB142V-5.08-4P, J4 DB142V-5.08-4P, K1 G5Q-1A4-DC24V, K2 G5Q-1A4-DC24V, K3 G5Q-1A4-DC24V, K4 G5Q-1A4-DC24V

Commit message: Replaced input terminal blocks for 3.5mm pitch.
Parts:
- J1, J2: Mfr DORABO -> Wago
Changed lines of the file:
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@@
 	(title_block
 		(title "4x 24V 8A Relay Module")
-		(date "2026-06-01")
+		(date "2026-06-02")
 		(rev "V1.1")
 	)
@@
 			)
 		)
-		(property "Mfr" "DORABO"
+		(property "Mfr" "Wago"
 			(at 29.21 74.93 0)
 			(hide yes)
@@
 			)
 		)
-		(property "Mfr" "DORABO"
+		(property "Mfr" "Wago"
 			(at 29.21 91.44 0)
 			(hide yes)
