File: V1/eumesmo-rl-4ch8a-v1.kicad_sch (KiCad schematic)
At the start: 24 parts, among them J1 250-202, J2 250-204, J3 DB142V-5.08-4P, J4 DB142V-5.08-4P, K1 G5Q-1A4-DC24V, K2 G5Q-1A4-DC24V, K3 G5Q-1A4-DC24V, K4 G5Q-1A4-DC24V

Commit message: Updated version numbers.
Other:
- title: 4x 24V 8A Relay Module -> eumesmo 4x 24V 8A Relay Module
Changed lines of the file:
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@@
 	(paper "A4")
 	(title_block
-		(title "4x 24V 8A Relay Module")
-		(date "2026-06-02")
-		(rev "V1.1")
+		(title "eumesmo 4x 24V 8A Relay Module")
+		(date "2026-06-13")
+		(rev "V1.2")
 	)
 	(text "CORRENTE NO LED\n24V - 2,85V = 21,15V\n21,15V / 10K = 2,11mA"
@@
 		)
 		(instances
-			(project "relay-24v-4ch-8a-v1"
+			(project "eumesmo-rl-4ch8a-v1"
 				(path "/57cfb5e7-a9ab-4784-80b3-e51e693f5cc8"
 					(reference "J1")
@@
 		)
 		(instances
-			(project "relay-24v-4ch-8a-v1"
+			(project "eumesmo-rl-4ch8a-v1"
 				(path "/57cfb5e7-a9ab-4784-80b3-e51e693f5cc8"
 					(reference "#PWR0103")
@@
 		)
 		(instances
-			(project "relay-24v-4ch-8a-v1"
+			(project "eumesmo-rl-4ch8a-v1"
 				(path "/57cfb5e7-a9ab-4784-80b3-e51e693f5cc8"
 					(reference "D7")
@@
 		)
 		(instances
-			(project "relay-24v-4ch-8a-v1"
+			(project "eumesmo-rl-4ch8a-v1"
 				(path "/57cfb5e7-a9ab-4784-80b3-e51e693f5cc8"
 					(reference "K3")
@@
 		)
 		(instances
-			(project "relay-24v-4ch-8a-v1"
+			(project "eumesmo-rl-4ch8a-v1"
 				(path "/57cfb5e7-a9ab-4784-80b3-e51e693f5cc8"
 					(reference "D2")
@@
 		)
 		(instances
-			(project "relay-24v-4ch-8a-v1"
+			(project "eumesmo-rl-4ch8a-v1"
 				(path "/57cfb5e7-a9ab-4784-80b3-e51e693f5cc8"
 					(reference "R1")
@@
 		)
 		(instances
-			(project "relay-24v-4ch-8a-v1"
+			(project "eumesmo-rl-4ch8a-v1"
 				(path "/57cfb5e7-a9ab-4784-80b3-e51e693f5cc8"
 					(reference "#PWR0101")
@@
 		)
 		(instances
-			(project "relay-24v-4ch-8a-v1"
+			(project "eumesmo-rl-4ch8a-v1"
 				(path "/57cfb5e7-a9ab-4784-80b3-e51e693f5cc8"
 					(reference "J2")
@@
 		)
 		(instances
-			(project "relay-24v-4ch-8a-v1"
+			(project "eumesmo-rl-4ch8a-v1"
 				(path "/57cfb5e7-a9ab-4784-80b3-e51e693f5cc8"
 					(reference "#FLG0101")
@@
 		)
 		(instances
-			(project "relay-24v-4ch-8a-v1"
+			(project "eumesmo-rl-4ch8a-v1"
 				(path "/57cfb5e7-a9ab-4784-80b3-e51e693f5cc8"
 					(reference "D5")
@@
 		)
 		(instances
-			(project "relay-24v-4ch-8a-v1"
+			(project "eumesmo-rl-4ch8a-v1"
 				(path "/57cfb5e7-a9ab-4784-80b3-e51e693f5cc8"
 					(reference "R3")
@@
 		)
 		(instances
-			(project "relay-24v-4ch-8a-v1"
+			(project "eumesmo-rl-4ch8a-v1"
 				(path "/57cfb5e7-a9ab-4784-80b3-e51e693f5cc8"
 					(reference "K4")
@@
 		)
 		(instances
-			(project "relay-24v-4ch-8a-v1"
+			(project "eumesmo-rl-4ch8a-v1"
 				(path "/57cfb5e7-a9ab-4784-80b3-e51e693f5cc8"
 					(reference "K1")
@@
 		)
 		(instances
-			(project "relay-24v-4ch-8a-v1"
+			(project "eumesmo-rl-4ch8a-v1"
 				(path "/57cfb5e7-a9ab-4784-80b3-e51e693f5cc8"
 					(reference "#PWR0105")
@@
 		)
 		(instances
-			(project "relay-24v-4ch-8a-v1"
+			(project "eumesmo-rl-4ch8a-v1"
 				(path "/57cfb5e7-a9ab-4784-80b3-e51e693f5cc8"
 					(reference "RV4")
@@
 		)
 		(instances
-			(project "relay-24v-4ch-8a-v1"
+			(project "eumesmo-rl-4ch8a-v1"
 				(path "/57cfb5e7-a9ab-4784-80b3-e51e693f5cc8"
 					(reference "R4")
@@
 		)
 		(instances
-			(project "relay-24v-4ch-8a-v1"
+			(project "eumesmo-rl-4ch8a-v1"
 				(path "/57cfb5e7-a9ab-4784-80b3-e51e693f5cc8"
 					(reference "D1")
@@
 		)
 		(instances
-			(project "relay-24v-4ch-8a-v1"
+			(project "eumesmo-rl-4ch8a-v1"
 				(path "/57cfb5e7-a9ab-4784-80b3-e51e693f5cc8"
 					(reference "RV2")
@@
 		)
 		(instances
-			(project "relay-24v-4ch-8a-v1"
+			(project "eumesmo-rl-4ch8a-v1"
 				(path "/57cfb5e7-a9ab-4784-80b3-e51e693f5cc8"
 					(reference "J4")
@@
 		)
 		(instances
-			(project "relay-24v-4ch-8a-v1"
+			(project "eumesmo-rl-4ch8a-v1"
 				(path "/57cfb5e7-a9ab-4784-80b3-e51e693f5cc8"
 					(reference "J3")
@@
 		)
 		(instances
-			(project "relay-24v-4ch-8a-v1"
+			(project "eumesmo-rl-4ch8a-v1"
 				(path "/57cfb5e7-a9ab-4784-80b3-e51e693f5cc8"
 					(reference "R2")
@@
 		)
 		(instances
-			(project "relay-24v-4ch-8a-v1"
+			(project "eumesmo-rl-4ch8a-v1"
 				(path "/57cfb5e7-a9ab-4784-80b3-e51e693f5cc8"
 					(reference "#PWR0104")
@@
 		)
 		(instances
-			(project "relay-24v-4ch-8a-v1"
+			(project "eumesmo-rl-4ch8a-v1"
 				(path "/57cfb5e7-a9ab-4784-80b3-e51e693f5cc8"
 					(reference "D8")
@@
 		)
 		(instances
-			(project "relay-24v-4ch-8a-v1"
+			(project "eumesmo-rl-4ch8a-v1"
 				(path "/57cfb5e7-a9ab-4784-80b3-e51e693f5cc8"
 					(reference "#PWR0102")
@@
 		)
 		(instances
-			(project "relay-24v-4ch-8a-v1"
+			(project "eumesmo-rl-4ch8a-v1"
 				(path "/57cfb5e7-a9ab-4784-80b3-e51e693f5cc8"
 					(reference "D6")
@@
 		)
 		(instances
-			(project "relay-24v-4ch-8a-v1"
+			(project "eumesmo-rl-4ch8a-v1"
 				(path "/57cfb5e7-a9ab-4784-80b3-e51e693f5cc8"
 					(reference "D3")
@@
 		)
 		(instances
-			(project "relay-24v-4ch-8a-v1"
+			(project "eumesmo-rl-4ch8a-v1"
 				(path "/57cfb5e7-a9ab-4784-80b3-e51e693f5cc8"
 					(reference "D4")
@@
 		)
 		(instances
-			(project "relay-24v-4ch-8a-v1"
+			(project "eumesmo-rl-4ch8a-v1"
 				(path "/57cfb5e7-a9ab-4784-80b3-e51e693f5cc8"
 					(reference "RV1")
@@
 		)
 		(instances
-			(project "relay-24v-4ch-8a-v1"
+			(project "eumesmo-rl-4ch8a-v1"
 				(path "/57cfb5e7-a9ab-4784-80b3-e51e693f5cc8"
 					(reference "RV3")
@@
 		)
 		(instances
-			(project "relay-24v-4ch-8a-v1"
+			(project "eumesmo-rl-4ch8a-v1"
 				(path "/57cfb5e7-a9ab-4784-80b3-e51e693f5cc8"
 					(reference "K2")
