File: V1/eumesmo-rl-4ch8a-v1.kicad_sch (KiCad schematic)
At the start: 24 parts, among them J1 250-202, J2 250-204, J3 DB142V-5.08-4P, J4 DB142V-5.08-4P, K1 G5Q-1A4-DC24V, K2 G5Q-1A4-DC24V, K3 G5Q-1A4-DC24V, K4 G5Q-1A4-DC24V

Commit message: Replaced 0603 size 10k resistors for 0805 size.
Parts:
- R1, R2, R3, R4: value 10k/100mW -> 10k/125mW; footprint Tales:R_0603_1608Metric -> Tales:R_0805_2012Metric; LCSC Part # C25804 -> C17414; Mfr UNI-ROYAL(Uniroyal Elec) -> Uniroyal; Mfr PN 0603WAF1002T5E -> 0805W8F1002T5E; Package 0603/1608 -> 0805/2012; Vendor PN C25804 -> C17414
Changed lines of the file:
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@@
 			)
 		)
-		(property "Value" "10k/100mW"
+		(property "Value" "10k/125mW"
 			(at 71.12 63.5 0)
 			(show_name no)
@@
 			)
 		)
-		(property "Footprint" "Tales:R_0603_1608Metric"
+		(property "Footprint" "Tales:R_0805_2012Metric"
 			(at 74.676 63.754 90)
 			(hide yes)
@@
 			)
 		)
-		(property "Mfr" "UNI-ROYAL(Uniroyal Elec)"
+		(property "Mfr" "Uniroyal"
 			(at 73.66 63.5 0)
 			(hide yes)
@@
 			)
 		)
-		(property "Mfr PN" "0603WAF1002T5E"
+		(property "Mfr PN" "0805W8F1002T5E"
 			(at 73.66 63.5 0)
 			(hide yes)
@@
 			)
 		)
-		(property "Vendor PN" "C25804"
+		(property "Vendor PN" "C17414"
 			(at 73.66 63.5 0)
 			(hide yes)
@@
 			)
 		)
-		(property "LCSC Part #" "C25804"
+		(property "LCSC Part #" "C17414"
 			(at 71.12 66.04 0)
 			(show_name no)
@@
 			)
 		)
-		(property "Package" "0603/1608"
+		(property "Package" "0805/2012"
 			(at 73.66 63.5 0)
 			(hide yes)
@@
 			)
 		)
-		(property "Value" "10k/100mW"
+		(property "Value" "10k/125mW"
 			(at 71.12 125.73 0)
 			(show_name no)
@@
 			)
 		)
-		(property "Footprint" "Tales:R_0603_1608Metric"
+		(property "Footprint" "Tales:R_0805_2012Metric"
 			(at 74.676 125.984 90)
 			(hide yes)
@@
 			)
 		)
-		(property "Mfr" "UNI-ROYAL(Uniroyal Elec)"
+		(property "Mfr" "Uniroyal"
 			(at 73.66 125.73 0)
 			(hide yes)
@@
 			)
 		)
-		(property "Mfr PN" "0603WAF1002T5E"
+		(property "Mfr PN" "0805W8F1002T5E"
 			(at 73.66 125.73 0)
 			(hide yes)
@@
 			)
 		)
-		(property "Vendor PN" "C25804"
+		(property "Vendor PN" "C17414"
 			(at 73.66 125.73 0)
 			(hide yes)
@@
 			)
 		)
-		(property "LCSC Part #" "C25804"
+		(property "LCSC Part #" "C17414"
 			(at 71.12 128.27 0)
 			(show_name no)
@@
 			)
 		)
-		(property "Package" "0603/1608"
+		(property "Package" "0805/2012"
 			(at 73.66 125.73 0)
 			(hide yes)
@@
 			)
 		)
-		(property "Value" "10k/100mW"
+		(property "Value" "10k/125mW"
 			(at 160.02 128.27 0)
 			(show_name no)
@@
 			)
 		)
-		(property "Footprint" "Tales:R_0603_1608Metric"
+		(property "Footprint" "Tales:R_0805_2012Metric"
 			(at 163.576 128.524 90)
 			(hide yes)
@@
 			)
 		)
-		(property "Mfr" "UNI-ROYAL(Uniroyal Elec)"
+		(property "Mfr" "Uniroyal"
 			(at 162.56 128.27 0)
 			(hide yes)
@@
 			)
 		)
-		(property "Mfr PN" "0603WAF1002T5E"
+		(property "Mfr PN" "0805W8F1002T5E"
 			(at 162.56 128.27 0)
 			(hide yes)
@@
 			)
 		)
-		(property "Vendor PN" "C25804"
+		(property "Vendor PN" "C17414"
 			(at 162.56 128.27 0)
 			(hide yes)
@@
 			)
 		)
-		(property "LCSC Part #" "C25804"
+		(property "LCSC Part #" "C17414"
 			(at 160.02 130.81 0)
 			(show_name no)
@@
 			)
 		)
-		(property "Package" "0603/1608"
+		(property "Package" "0805/2012"
 			(at 162.56 128.27 0)
 			(hide yes)
@@
 			)
 		)
-		(property "Value" "10k/100mW"
+		(property "Value" "10k/125mW"
 			(at 160.02 66.04 0)
 			(show_name no)
@@
 			)
 		)
-		(property "Footprint" "Tales:R_0603_1608Metric"
+		(property "Footprint" "Tales:R_0805_2012Metric"
 			(at 163.576 66.294 90)
 			(hide yes)
@@
 			)
 		)
-		(property "Mfr" "UNI-ROYAL(Uniroyal Elec)"
+		(property "Mfr" "Uniroyal"
 			(at 162.56 66.04 0)
 			(hide yes)
@@
 			)
 		)
-		(property "Mfr PN" "0603WAF1002T5E"
+		(property "Mfr PN" "0805W8F1002T5E"
 			(at 162.56 66.04 0)
 			(hide yes)
@@
 			)
 		)
-		(property "Vendor PN" "C25804"
+		(property "Vendor PN" "C17414"
 			(at 162.56 66.04 0)
 			(hide yes)
@@
 			)
 		)
-		(property "LCSC Part #" "C25804"
+		(property "LCSC Part #" "C17414"
 			(at 160.02 68.58 0)
 			(show_name no)
@@
 			)
 		)
-		(property "Package" "0603/1608"
+		(property "Package" "0805/2012"
 			(at 162.56 66.04 0)
 			(hide yes)
