File: V1/eumesmo-rl-4ch8a-v1.kicad_pcb (KiCad board)
At the start: 2 copper layers, 53 x 67.8 mm, 25 parts, among them J1 250-202, J2 250-204, J3 DB142V-5.08-4P, J4 DB142V-5.08-4P, K1 G5Q-1A4-DC24V, K2 G5Q-1A4-DC24V, K3 G5Q-1A4-DC24V, K4 G5Q-1A4-DC24V

Commit message: Replaced 0603 size 10k resistors for 0805 size.
Parts:
- R1, R2, R3, R4: value 10k/100mW -> 10k/125mW; footprint Tales:R_0603_1608Metric -> Tales:R_0805_2012Metric
- moved R1 1.50 mm to (148.0, 65.5)
- moved R2 1.00 mm to (148.0, 67.5)
- moved R3 0.50 mm to (148.0, 69.5)
Routing:
- net +24V: track 117.5 -> 119.6 mm
- net /LED1: track 20.3 -> 20.8 mm
